File: PCB design/Aura-Board/Aura-Board.kicad_pcb (KiCad board)
At the start: 2 copper layers, 144.5 x 124.7 mm, 8 parts, among them J1 4-digit 7 segment display, J2 Touch_Sensor, U1 ESP32-DEVKIT-V1, U2 DM-OLED096-636, U3 OC09600

Commit message: update PCB design files
Parts:
- added D1: LED, PCM_4ms_LED:LED_5mm_RightAngle, F.Cu at (98.5, 43.0)
- added D2: LED, PCM_4ms_LED:LED_5mm_RightAngle, F.Cu at (98.0, 73.0)
- added D3: LED, PCM_4ms_LED:LED_5mm_RightAngle, F.Cu at (95.5, 93.0)
- added ST1: Standoff, PCM_SparkFun-Hardware:Standoff_Connected, F.Cu at (92.0, 34.0)
- added ST2: Standoff, PCM_SparkFun-Hardware:Standoff_Connected, F.Cu at (272.5, 36.5)
- added ST3: Standoff, PCM_SparkFun-Hardware:Standoff_Connected, F.Cu at (90.0, 114.0)
- added ST4: Standoff, PCM_SparkFun-Hardware:Standoff_Connected, F.Cu at (274.0, 113.5)
- moved J1 113.3 mm to (199.0, 89.4), turned to 0 degrees
- moved J2 77.7 mm to (139.5, 86.0)
- moved U2 75.7 mm to (173.5, 97.5)
- moved R3 45.1 mm to (114.0, 93.0), turned to 180 degrees
- moved U3 40.8 mm to (242.1, 51.6), turned to 180 degrees
- moved R2 31.5 mm to (113.5, 76.0), turned to 180 degrees
- moved U1 26.6 mm to (175.5, 49.5), turned to 90 degrees
- moved R1 5.97 mm to (113.0, 45.0), turned to 180 degrees
Routing:
- net VCC: track 0.00 -> 389.7 mm
- net GND: track 267.5 -> 646.8 mm
- net Net-(J2-Pin_1): track 0.00 -> 240.5 mm
- net Net-(U1-D4): track 0.00 -> 97.1 mm
- net Net-(U1-D25): track 0.00 -> 83.0 mm
- net Net-(U1-D5): track 0.00 -> 75.0 mm
- net Net-(U1-D2): track 0.00 -> 60.2 mm
- net Net-(J1-Pin_1): track 0.00 -> 52.3 mm
- net Net-(J1-Pin_2): track 0.00 -> 47.1 mm
- net Net-(U1-D26): track 43.4 -> 79.8 mm
- net 22: track 0.00 -> 31.1 mm
- net 21: track 0.00 -> 28.2 mm
- net Net-(D3-Pad1): track 0.00 -> 13.0 mm
- net Net-(D2-Pad1): track 0.00 -> 10.2 mm
- net Net-(D1-Pad1): track 0.00 -> 8.76 mm
Other:
- board size 144.5 x 124.7 mm -> 192 x 89 mm
